Commit message: add realsense camera

File: src/simulation_bringup/urdf/sensebeetle_original.xacro (robot description, xacro)
@@ -160,4 +160,31 @@
     </inertial>
   </link>
+  <!-- Depth Camera -->
+  <link name="depth_camera_link">
+    <visual>
+      <geometry>
+        <box size="0.05 0.05 0.1"/>
+      </geometry>
+      <origin xyz="0 0 0" rpy="0 0 0"/>
+      <material name="blue">
+        <color rgba="0 0 1 1"/>
+      </material>
+    </visual>
+    <collision>
+      <geometry>
+        <box size="0.05 0.05 0.1"/>
+      </geometry>
+    </collision>
+    <inertial>
+      <mass value="0.1"/>
+      <origin xyz="0 0 0" rpy="0 0 0"/>
+      <inertia ixx="0.0001" ixy="0" ixz="0" iyy="0.0001" iyz="0" izz="0.0001"/>
+    </inertial>
+  </link>
+  <joint name="base_to_depth_camera" type="fixed">
+    <parent link="base_link"/>
+    <child link="depth_camera_link"/>
+    <origin xyz="0 0 0.2" rpy="0 0 0"/>
+  </joint>
   <gazebo reference="base_link">
     <material>Gazebo/Purple</material>
@@ -180,4 +207,40 @@
   <gazebo reference="livox_frame">
     <material>Gazebo/LightBlueLaser</material>
+  </gazebo>
+  <!-- 深度相机传感器 - 使用正确的深度相机插件 -->
+  <gazebo reference="depth_camera_link">
+    <material>Gazebo/Blue</material>
+    <sensor name="depth_camera" type="depth">
+      <always_on>true</always_on>
+      <update_rate>5</update_rate>
+      <visualize>false</visualize>
+      <camera>
+        <horizontal_fov>1.047</horizontal_fov>
+        <image>
+          <width>640</width>
+          <height>480</height>
+          <format>R8G8B8</format>
+        </image>
+        <clip>
+          <near>0.1</near>
+          <far>10.0</far>
+        </clip>
+      </camera>
+      <plugin name="depth_camera_controller" filename="libgazebo_ros_camera.so">
+        <ros>
+          <namespace>$(arg robot_namespace)</namespace>
+          <remapping>depth/image_raw:=camera/depth/image_raw</remapping>
+          <remapping>depth/camera_info:=camera/depth/camera_info</remapping>
+          <remapping>image_raw:=camera/image_raw</remapping>
+          <remapping>camera_info:=camera/camera_info</remapping>
+          <remapping>points:=camera/points</remapping>
+        </ros>
+        <camera_name>camera</camera_name>
+        <frame_name>$(arg robot_namespace)/depth_camera_link</frame_name>
+        <hack_baseline>0.07</hack_baseline>
+        <min_depth>0.1</min_depth>
+        <max_depth>10.0</max_depth>
+      </plugin>
+    </sensor>
   </gazebo>
   <!-- Drive controller plugin-->
